Commit message: implemented moveit setup assistant

File: src/arm_description/urdf/arm.xacro (robot description, xacro)
@@ -11,6 +11,7 @@
         <collision>
             <geometry>
-                <origin xyz="0 0 0.05" rpy="0 0 0"/>
+                <box size= "0.4 0.4 0.1"/>
             </geometry>
+            <origin xyz="0 0 0.05" rpy="0 0 0"/>
         </collision>
     </link>
@@ -23,4 +24,10 @@
             <material name="blue"/>
         </visual>
+        <collision>
+            <geometry>
+                <box size="0.2 0.2 0.5"/>
+            </geometry>
+            <origin xyz="0 0 0.25" rpy="0 0 0"/>
+        </collision>
     </link>
     <link name="shoulder_link">
@@ -32,4 +39,10 @@
             <material name="grey"/>
         </visual>
+        <collision>
+            <geometry>
+                <box size="0.1 0.1 0.6"/>
+            </geometry>
+            <origin xyz="0 0 0.3" rpy="0 0 0"/>
+        </collision>
     </link>
     <link name="elbow_link">
@@ -41,4 +54,10 @@
             <material name="blue"/>
         </visual>
+        <collision>
+            <geometry>
+                <box size="0.1 0.1 0.1"/>
+            </geometry>
+            <origin xyz="0 0 0.05" rpy="0 0 0"/>
+        </collision>
     </link>
     <link name="forearm_link">
@@ -50,4 +69,10 @@
             <material name="grey"/>
         </visual>
+        <collision>
+            <geometry>
+                <box size="0.1 0.1 0.6"/>
+            </geometry>
+            <origin xyz="0 0 0.3" rpy="0 0 0"/>
+        </collision>
     </link>
     <link name="wrist_link">
@@ -59,4 +84,10 @@
             <material name="blue"/>
         </visual>
+        <collision>
+            <geometry>
+                <box size="0.1 0.1 0.05"/>
+            </geometry>
+            <origin xyz="0 0 0.025" rpy="0 0 0"/>
+        </collision>
     </link>
     <link name="hand_link">
@@ -68,4 +99,10 @@
             <material name="grey"/>
         </visual>
+        <collision>
+            <geometry>
+                <box size="0.1 0.1 0.02"/>
+            </geometry>
+            <origin xyz="0 0 0.01" rpy="0 0 0"/>
+        </collision>
     </link>
     <link name="tool_link"/>
@@ -105,10 +142,10 @@
         <limit effort="1000.0" velocity="1.0" lower="-1.57" upper="1.57"/>
     </joint>
-    <joint name="hand_to_wrist_joint" type="revolute">
+    <joint name="hand_to_wrist_joint" type="continuous">
         <parent link="wrist_link"/>
         <child link="hand_link"/>
         <origin xyz="0 0 0.05" rpy="0 0 0"/>
         <axis xyz="0 0 1"/>
-        <limit effort="1000.0" velocity="1.0" lower="-3.14" upper="3.14"/>
+        <!-- <limit effort="1000.0" velocity="1.0" lower="-3.14" upper="3.14"/> -->
     </joint>
     <joint name="tool_to_hand_joint" type="fixed">
